File: Single_transistor_AMP/Single_transistor_AMP.sch (KiCad schematic (older format))
At the start: 10 parts, among them P1 Signal_In, P2 Signal_Out, Q1 BC548

Commit message: Work after VII lecture
Parts:
- added P3: PWR_Con, Connector:Banana_Jack_2Pin, symbol PWR_Con:PWR_Con
Connections:
- net +12V: now also P3.1
- new net Earth: P3.2
Changed lines of the file:
@@
 F 0 "#PWR03" H 6340 3300 50  0001 C CNN
 F 1 "+12V" H 6355 3623 50  0000 C CNN
-F 2 "Connector_Wire:SolderWire-0.5sqmm_1x01_D0.9mm_OD2.1mm" H 6340 3450 50  0001 C CNN
+F 2 "Connector:Banana_Jack_2Pin" H 6340 3450 50  0001 C CNN
 F 3 "" H 6340 3450 50  0001 C CNN
 	1    6340 3450
@@
 F 0 "#PWR02" H 6100 4450 50  0001 C CNN
 F 1 "GND" H 6105 4527 50  0000 C CNN
-F 2 "" H 6100 4700 50  0001 C CNN
+F 2 "Connector:Banana_Jack_1Pin" H 6100 4700 50  0001 C CNN
 F 3 "" H 6100 4700 50  0001 C CNN
 	1    6100 4700
@@
 Wire Wire Line
 	4400 4100 4510 4100
+$Comp
+L PWR_Con:PWR_Con P3
+U 1 1 5FD937E3
+P 7310 4600
+F 0 "P3" H 7388 4641 50  0000 L CNN
+F 1 "PWR_Con" H 7388 4550 50  0000 L CNN
+F 2 "Connector:Banana_Jack_2Pin" H 7260 4600 50  0001 C CNN
+F 3 "" H 7260 4600 50  0001 C CNN
+	1    7310 4600
+	1    0    0    -1
+$EndComp
+$Comp
+L power:Earth #PWR0101
+U 1 1 5FD9447D
+P 7080 4650
+F 0 "#PWR0101" H 7080 4400 50  0001 C CNN
+F 1 "Earth" H 7080 4500 50  0001 C CNN
+F 2 "" H 7080 4650 50  0001 C CNN
+F 3 "~" H 7080 4650 50  0001 C CNN
+	1    7080 4650
+	1    0    0    -1
+$EndComp
+Wire Wire Line
+	7080 4650 7160 4650
+$Comp
+L power:+12V #PWR0102
+U 1 1 5FD95123
+P 7080 4550
+F 0 "#PWR0102" H 7080 4400 50  0001 C CNN
+F 1 "+12V" H 7095 4723 50  0000 C CNN
+F 2 "" H 7080 4550 50  0001 C CNN
+F 3 "" H 7080 4550 50  0001 C CNN
+	1    7080 4550
+	1    0    0    -1
+$EndComp
+Wire Wire Line
+	7080 4550 7160 4550
 $EndSCHEMATC
