File: Single_transistor_AMP/Single_transistor_AMP.kicad_pcb (KiCad board)
At the start: 2 copper layers, 10 parts, among them P1 Signal_In, P2 Signal_Out, Q1 BC548

Commit message: Work after V lecture
Parts:
- removed C1, C3: 20uF, Capacitor_THT:C_Disc_D5.0mm_W2.5mm_P5.00mm
- removed C2: 50uF, Capacitor_THT:C_Disc_D5.0mm_W2.5mm_P5.00mm
- removed P1: Signal_In, Connector_Wire:SolderWire-0.5sqmm_1x02_P4.6mm_D0.9mm_OD2.1mm
- removed P2: Signal_Out, Connector_Wire:SolderWire-0.5sqmm_1x02_P4.6mm_D0.9mm_OD2.1mm
- removed Q1: BC548, Package_TO_SOT_THT:TO-92_Inline
- removed R1: 22k, Resistor_THT:R_Axial_DIN0204_L3.6mm_D1.6mm_P5.08mm_Horizontal
- removed R2: 6.8k, Resistor_THT:R_Axial_DIN0204_L3.6mm_D1.6mm_P7.62mm_Horizontal
- removed R3: 4.7k, Resistor_THT:R_Axial_DIN0204_L3.6mm_D1.6mm_P7.62mm_Horizontal
- removed R4: 1.8k, Resistor_THT:R_Axial_DIN0204_L3.6mm_D1.6mm_P7.62mm_Horizontal
Other:
- net class Diff added: clearance 0.125, trace_width 1.15, via_dia 0.8, via_drill 0.4
- net class Power added: clearance 0.8, trace_width 0.5, via_dia 1, via_drill 0.8

Commit message: Work after VII lecture
Parts:
- added C1: 20uF, Capacitor_THT:C_Disc_D5.0mm_W2.5mm_P5.00mm, F.Cu at (136.2, 95.3)
- added C2: 50uF, Capacitor_THT:C_Disc_D5.0mm_W2.5mm_P5.00mm, F.Cu at (160.9, 90.6)
- added C3: 20uF, Capacitor_THT:C_Disc_D5.0mm_W2.5mm_P5.00mm, F.Cu at (160.9, 104.5)
- added P1: Signal_In, Connector_Wire:SolderWire-0.5sqmm_1x02_P4.6mm_D0.9mm_OD2.1mm, F.Cu at (131.3, 100.0)
- added P2: Signal_Out, Connector_Wire:SolderWire-0.5sqmm_1x02_P4.6mm_D0.9mm_OD2.1mm, F.Cu at (163.9, 100.0)
- added P3: PWR_Con, Connector:Banana_Jack_2Pin, F.Cu at (132.9, 113.0)
- added Q1: BC548, Package_TO_SOT_THT:TO-92_Inline, F.Cu at (150.9, 98.8)
- added R1: 22k, Resistor_THT:R_Axial_DIN0204_L3.6mm_D1.6mm_P5.08mm_Horizontal, F.Cu at (140.5, 100.4)
- added R2: 6.8k, Resistor_THT:R_Axial_DIN0204_L3.6mm_D1.6mm_P7.62mm_Horizontal, F.Cu at (144.8, 93.8)
- added R3: 4.7k, Resistor_THT:R_Axial_DIN0204_L3.6mm_D1.6mm_P7.62mm_Horizontal, F.Cu at (159.5, 93.9)
- added R4: 1.8k, Resistor_THT:R_Axial_DIN0204_L3.6mm_D1.6mm_P7.62mm_Horizontal, F.Cu at (155.9, 93.9)
Other:
- board outline added: 47.9 x 32.6 mm

Commit message: Work after IX lecture
Parts:
- moved P1 0.36 mm to (131.3, 100.4)
- moved P3 0.31 mm to (133.0, 113.3)
- moved R1 0.15 mm to (140.6, 100.4)
- moved C1 0.05 mm to (136.2, 95.3)
Routing:
- net +12V: track 0.00 -> 68.1 mm
- net Net-(C1-Pad1): track 0.00 -> 17.8 mm
- net Net-(C3-Pad2): track 0.00 -> 13.7 mm
- net Net-(C2-Pad2): track 0.00 -> 9.24 mm
- net Net-(C3-Pad1): track 0.00 -> 5.72 mm
- net Net-(C1-Pad2): track 0.00 -> 4.97 mm
- added copper zone on B.Cu, net GND
- added copper zone on F.Cu, net GND
